Commit message: initial commit

File: urdf/anymal_main.xacro (robot description, xacro)
@@ -1,10 +1,9 @@
 <?xml version="1.0"?>
 <robot xmlns:xacro="http://www.ros.org/wiki/xacro"  name="anymal">
-    <material name="orange">
-        <color rgba="1 0.3 0.1 1"/>
-    </material>
-    <material name="red">
-        <color rgba="1 0 0 1"/>
-    </material>
+    <xacro:arg name="remove_shank_collisions" default="False"/>
+    <xacro:property name="remove_shank_collisions" default="$(arg remove_shank_collisions)"/>
     <xacro:include filename="anymal.urdf.xacro" />
+    <xacro:include filename="anymal_gazebo.xacro" />
+    <xacro:include filename="materials.xacro" />
+    <xacro:include filename="inertial_macros.xacro" />
 </robot>

Commit message: added lidar simulation xacro

File: urdf/anymal_main.xacro (robot description, xacro)
@@ -7,3 +7,4 @@
     <xacro:include filename="materials.xacro" />
     <xacro:include filename="inertial_macros.xacro" />
+    <xacro:include filename="lidar.xacro" />
 </robot>

File: urdf/lidar.xacro (robot description, xacro)
@@ -1,5 +1,5 @@
 <?xml version="1.0"?>
 <robot xmlns:xacro="http://www.ros.org/wiki/xacro" >
-    <joint name="laser_joint" type="fixed">
+    <!-- <joint name="laser_joint" type="fixed">
         <parent link="base"/>
         <child link="laser_frame"/>
@@ -21,6 +21,6 @@
             <origin xyz="0 0 0" rpy="0 0 0"/>
         </xacro:inertial_cylinder>
-    </link>
-    <gazebo reference="laser_frame">
+    </link> -->
+    <gazebo reference="lidar">
         <material>Gazebo/Red</material>
         <sensor name="laser" type="ray">
@@ -43,9 +43,8 @@
             <plugin name="laser_controller" filename="libgazebo_ros_ray_sensor.so">
                 <ros>
-                    <!-- <argument>~/out:=scan</argument> -->
                     <argument>--ros-args --remap ~/out:=scan</argument>
                 </ros>
                 <output_type>sensor_msgs/LaserScan</output_type>
-                <frame_name>laser_frame</frame_name>
+                <frame_name>lidar</frame_name>
             </plugin>
         </sensor>
