Commit message: added p3d section

File: urdf/lidar.xacro (robot description, xacro)
@@ -1,25 +1,17 @@
 <?xml version="1.0"?>
 <robot xmlns:xacro="http://www.ros.org/wiki/xacro" >
-    <!-- <joint name="laser_joint" type="fixed">
-        <parent link="base"/>
-        <child link="laser_frame"/>
-        <origin xyz="0.1 0 0.175" rpy="0 0 0"/>
-    </joint>
-    <link name="laser_frame">
-        <visual>
-            <geometry>
-                <cylinder radius="0.05" length="0.04"/>
-            </geometry>
-            <material name="red"/>
-        </visual>
-        <collision>
-            <geometry>
-                <cylinder radius="0.05" length="0.04"/>
-            </geometry>
-        </collision>
-        <xacro:inertial_cylinder mass="0.1" length="0.04" radius="0.05">
-            <origin xyz="0 0 0" rpy="0 0 0"/>
-        </xacro:inertial_cylinder>
-    </link> -->
+    <gazebo>
+        <plugin filename="libgazebo_ros_p3d.so" name="p3d_base_controller">
+        <ros>
+            <argument>odom:=odom/ground_truth</argument>
+        </ros>
+        <body_name>base</body_name>
+        <frame_name>map</frame_name>
+        <update_rate>100.0</update_rate>
+        <xyz_offset>-0.364 0.0 0.0</xyz_offset>
+        <rpy_offset>0 0 0</rpy_offset>
+        <gaussian_noise>0.0</gaussian_noise>
+        </plugin>
+    </gazebo>
     <gazebo reference="lidar">
         <material>Gazebo/Red</material>
@@ -37,6 +29,6 @@
                 </scan>
                 <range>
-                    <min>0.3</min>
-                    <max>12</max>
+                    <min>0.8</min>
+                    <max>20</max>
                 </range>
             </ray>

Commit message: added lidar macro

File: urdf/lidar.xacro (robot description, xacro)
@@ -8,37 +8,37 @@
         <body_name>base</body_name>
         <frame_name>map</frame_name>
-        <update_rate>100.0</update_rate>
-        <xyz_offset>-0.364 0.0 0.0</xyz_offset>
+        <update_rate>10.0</update_rate>
+        <xyz_offset>0.0 0.0 -.5</xyz_offset>
         <rpy_offset>0 0 0</rpy_offset>
-        <gaussian_noise>0.0</gaussian_noise>
         </plugin>
     </gazebo>
-    <gazebo reference="lidar">
-        <material>Gazebo/Red</material>
-        <sensor name="laser" type="ray">
-            <pose> 0 0 0 0 0 0 </pose>
-            <visualize>true</visualize>
-            <update_rate>10</update_rate>
-            <ray>
-                <scan>
-                    <horizontal>
-                        <samples>360</samples>
-                        <min_angle>-3.14</min_angle>
-                        <max_angle>3.14</max_angle>
-                    </horizontal>
-                </scan>
-                <range>
-                    <min>0.8</min>
-                    <max>20</max>
-                </range>
-            </ray>
-            <plugin name="laser_controller" filename="libgazebo_ros_ray_sensor.so">
-                <ros>
-                    <argument>--ros-args --remap ~/out:=scan</argument>
-                </ros>
-                <output_type>sensor_msgs/LaserScan</output_type>
-                <frame_name>lidar</frame_name>
-            </plugin>
-        </sensor>
-    </gazebo>
+    <xacro:macro name="lidar_macro" params="max_range samples">
+        <gazebo reference="base">
+            <sensor name="laser" type="ray">
+                <pose> 0 0 .2 0 0 0 </pose>
+                <visualize>false</visualize>
+                <update_rate>10</update_rate>
+                <ray>
+                    <scan>
+                        <horizontal>
+                            <samples>${samples}</samples>
+                            <min_angle>-3.14</min_angle>
+                            <max_angle>3.14</max_angle>
+                        </horizontal>
+                    </scan>
+                    <range>
+                        <min>0.45</min>
+                        <max>${max_range}</max>
+                    </range>
+                </ray>
+                <plugin name="laser_controller_${max_range}_${samples}" filename="libgazebo_ros_ray_sensor.so">
+                    <output_type>sensor_msgs/LaserScan</output_type>
+                    <frame_name>lidar_frame</frame_name>
+                </plugin>
+            </sensor>
+        </gazebo>
+    </xacro:macro>
+    <xacro:lidar_macro max_range="5" samples="360"></xacro:lidar_macro>
+    <xacro:lidar_macro max_range="10" samples="360"></xacro:lidar_macro>
+    <xacro:lidar_macro max_range="15" samples="360"></xacro:lidar_macro>
 </robot>
