Commit message: converted package for ros noetic

File: urdf/anymal_floating_base.urdf (robot description, URDF)
Before this commit: robot anymal, 78 links, 77 joints
Links:
- added link floating_base
- link LF_FOOT: geometry collision cylinder length=0.282504 radius=0.0175; collision sphere radius=0.03
- link LF_HAA: geometry visual mesh filename=package://anymal_c_simple_description/meshes/drive.dae scale=1.0 1.0 1.0
- link LF_HFE: geometry collision cylinder length=0.14 radius=0.05; visual mesh filename=package://anymal_c_simple_description/meshes/drive.dae scale=1.0 1.0 1.0
- link LF_KFE: geometry collision cylinder length=0.14 radius=0.05; visual mesh filename=package://anymal_c_simple_description/meshes/drive.dae scale=1.0 1.0 1.0
- link LF_hip_fixed: geometry visual mesh filename=package://anymal_c_simple_description/meshes/hip_l.dae scale=1.0 1.0 1.0
- link LF_shank_fixed: geometry collision box size=0.114998 0.0675 0.04; collision cylinder length=0.04 radius=0.06
- link LF_thigh_fixed: geometry collision box size=0.075 0.06 0.282627; collision cylinder length=0.08 radius=0.065
- link LH_FOOT: geometry collision cylinder length=0.282504 radius=0.0175; collision sphere radius=0.03
- link LH_HAA: geometry visual mesh filename=package://anymal_c_simple_description/meshes/drive.dae scale=1.0 1.0 1.0
- link LH_HFE: geometry collision cylinder length=0.14 radius=0.05; visual mesh filename=package://anymal_c_simple_description/meshes/drive.dae scale=1.0 1.0 1.0
- link LH_KFE: geometry collision cylinder length=0.14 radius=0.05; visual mesh filename=package://anymal_c_simple_description/meshes/drive.dae scale=1.0 1.0 1.0
- link LH_hip_fixed: geometry visual mesh filename=package://anymal_c_simple_description/meshes/hip_r.dae scale=1.0 1.0 1.0
- link LH_shank_fixed: geometry collision box size=0.114998 0.0675 0.04; collision cylinder length=0.04 radius=0.06
- link LH_thigh_fixed: geometry collision box size=0.075 0.06 0.282627; collision cylinder length=0.08 radius=0.065
- link RF_FOOT: geometry collision cylinder length=0.282504 radius=0.0175; collision sphere radius=0.03
- link RF_HAA: geometry visual mesh filename=package://anymal_c_simple_description/meshes/drive.dae scale=1.0 1.0 1.0
- link RF_HFE: geometry collision cylinder length=0.14 radius=0.05; visual mesh filename=package://anymal_c_simple_description/meshes/drive.dae scale=1.0 1.0 1.0
- link RF_KFE: geometry collision cylinder length=0.14 radius=0.05; visual mesh filename=package://anymal_c_simple_description/meshes/drive.dae scale=1.0 1.0 1.0
- link RF_hip_fixed: geometry visual mesh filename=package://anymal_c_simple_description/meshes/hip_r.dae scale=1.0 1.0 1.0
- link RF_shank_fixed: geometry collision box size=0.114998 0.0675 0.04; collision cylinder length=0.04 radius=0.06
- link RF_thigh_fixed: geometry collision box size=0.075 0.06 0.282627; collision cylinder length=0.08 radius=0.065
- link RH_FOOT: geometry collision cylinder length=0.282504 radius=0.0175; collision sphere radius=0.03
- link RH_HAA: geometry visual mesh filename=package://anymal_c_simple_description/meshes/drive.dae scale=1.0 1.0 1.0
- link RH_HFE: geometry collision cylinder length=0.14 radius=0.05; visual mesh filename=package://anymal_c_simple_description/meshes/drive.dae scale=1.0 1.0 1.0
- link RH_KFE: geometry collision cylinder length=0.14 radius=0.05; visual mesh filename=package://anymal_c_simple_description/meshes/drive.dae scale=1.0 1.0 1.0
- link RH_hip_fixed: geometry visual mesh filename=package://anymal_c_simple_description/meshes/hip_l.dae scale=1.0 1.0 1.0
- link RH_shank_fixed: geometry collision box size=0.114998 0.0675 0.04; collision cylinder length=0.04 radius=0.06
- link RH_thigh_fixed: geometry collision box size=0.075 0.06 0.282627; collision cylinder length=0.08 radius=0.065
- link base: geometry collision box size=0.58 0.14 0.18; collision cylinder length=0.145 radius=0.09
- link battery: geometry visual mesh filename=package://anymal_c_simple_description/meshes/battery.dae scale=1.0 1.0 1.0
- link bottom_shell: geometry visual mesh filename=package://anymal_c_simple_description/meshes/bottom_shell.d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 scale=1.0 1.0 1.0
- link depth_camera_front_camera: geometry visual mesh filename=package://anymal_c_simple_description/meshes/depth_camera.d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 scale=1.0 1.0 1.0
- link depth_camera_left_camera: geometry visual mesh filename=package://anymal_c_simple_description/meshes/depth_camera.d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 scale=1.0 1.0 1.0
- link depth_camera_rear_camera: geometry visual mesh filename=package://anymal_c_simple_description/meshes/depth_camera.d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 scale=1.0 1.0 1.0
- link depth_camera_right_camera: geometry visual mesh filename=package://anymal_c_simple_description/meshes/depth_camera.d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 scale=1.0 1.0 1.0
- link face_front: geometry collision box size=0.11 0.14 0.18; collision cylinder length=0.11 radius=0.09
- link face_rear: geometry collision box size=0.11 0.14 0.18; collision cylinder length=0.11 radius=0.09
- link handle: geometry visual mesh filename=package://anymal_c_simple_description/meshes/handle.dae scale=1.0 1.0 1.0
- link hatch: geometry visual mesh filename=package://anymal_c_simple_description/meshes/hatch.dae scale=1.0 1.0 1.0
- link lidar: geometry visual mesh filename=package://anymal_c_simple_description/meshes/lidar.dae
- link lidar_cage: geometry collision cylinder length=0.12 radius=0.07; visual mesh filename=package://anymal_c_simple_description/meshes/lidar_cage.dae scale=1.0 1.0 1.0
- link remote: geometry visual mesh filename=package://anymal_c_simple_description/meshes/remote.dae scale=1.0 1.0 1.0
- link top_shell: geometry visual mesh filename=package://anymal_c_simple_description/meshes/top_shell.dae scale=1.0 1.0 1.0
- link wide_angle_camera_front_camera: geometry visual mesh filename=package://anymal_c_simple_description/meshes/wide_angle_cam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 scale=1.0 1.0 1.0
- link wide_angle_camera_rear_camera: geometry visual mesh filename=package://anymal_c_simple_description/meshes/wide_angle_cam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 scale=1.0 1.0 1.0
Joints:
- added joint virtual: type floating, parent floating_base, child base, origin xyz=0 0 0 rpy=0 0 0, axis 0 0 1
